Commit message: Update ND_alternative_V21.SLDASM.urdf
Changed name to nemo1

File: nemo1/urdf/ND_alternative_V21.SLDASM.urdf (robot description, URDF)
Before this commit: robot ND_alternative_V21.SLDASM, 8 links, 7 joints
Links:
- link EE: geometry collision mesh filename=package://nemo1/meshes/EE.STL; visual mesh filename=package://nemo1/meshes/EE.STL
- link base_link: geometry collision mesh filename=package://nemo1/meshes/base_link.STL; visual mesh filename=package://nemo1/meshes/base_link.STL
- link link_1: geometry collision mesh filename=package://nemo1/meshes/link_1.STL; visual mesh filename=package://nemo1/meshes/link_1.STL
- link link_2: geometry collision mesh filename=package://nemo1/meshes/link_2.STL; visual mesh filename=package://nemo1/meshes/link_2.STL
- link link_3: geometry collision mesh filename=package://nemo1/meshes/link_3.STL; visual mesh filename=package://nemo1/meshes/link_3.STL
- link link_4: geometry collision mesh filename=package://nemo1/meshes/link_4.STL; visual mesh filename=package://nemo1/meshes/link_4.STL
- link link_5: geometry collision mesh filename=package://nemo1/meshes/link_5.STL; visual mesh filename=package://nemo1/meshes/link_5.STL
- link link_6: geometry collision mesh filename=package://nemo1/meshes/link_6.STL; visual mesh filename=package://nemo1/meshes/link_6.STL
